File: _autosave-flyback1.kicad_sch (KiCad schematic)
At the start: 38 parts, among them IC1 INN3649C-H606-TL, J2 Conn_01x02_Socket, Q1 100V, T1 P0544NL

Commit message: schematic is done
Parts:
- removed DC: 100-600 V, symbol Device:Battery_Cell
- added BT1: 100-600V, symbol Device:Battery
- renumbered R to R4
Connections:
- net Earth: now also BT1.2 (-)
- net VCC: now also BT1.1 (+)
Other:
- moved on the sheet: C13, C15, C16, C2.1, C2.2, C5, C6, C9, D2, D3, J2, R15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
