File: flyback1.kicad_sch (KiCad schematic)
At the start: 52 parts, among them IC1 INN3649C-H606-TL, J1 Conn_02x08_Odd_Even, J2 Conn_02x06_Odd_Even, Q1 100V, T1 P0544NL

Commit message: pcb is organized
Parts:
- added C1: 680p, Capacitor_THT:C_Disc_D8.0mm_W5.0mm_P10.00mm, symbol Device:C
- C2.2: footprint aaa:B58031U9254M062 -> Capacitor_THT:C_Disc_D8.0mm_W5.0mm_P10.00mm
Connections:
- net OUT2 is gone; now on net GND2: C15.2, C16.2, C17.2, C18.2, J2.10 (Pin_10), J2.11 (Pin_11), J2.12 (Pin_12), J2.7 (Pin_7), J2.8 (Pin_8), J2.9 (Pin_9), R13.2, R14.2
- net T6: now also C2.1.1, C2.2.1, C2.3.1, C2.4.1, J1.1 (Pin_1), J1.2 (Pin_2), J1.3 (Pin_3), J1.4 (Pin_4), J1.5 (Pin_5), J1.6 (Pin_6), C1.1
- net GND1: now reaches C2.1.2, C2.2.2, C2.3.2, C2.4.2, J1.11 (Pin_11), J1.12 (Pin_12), J1.13 (Pin_13), J1.14 (Pin_14), J1.15 (Pin_15), J1.16 (Pin_16)
- net GND1: now also C5.2, C6.2, D1.2 (A), IC1.16 (S), IC1.24 (D), T1.8, T1.9
- net GND renamed GND2
- net GND2: now also C1.2; no longer C5.2, C6.2, D1.2 (A), IC1.16 (S), IC1.24 (D), T1.8, T1.9
Other:
- moved on the sheet: T1

Commit message: tracks drawn
Parts:
- Q1: value 100V -> 150V
Connections:
- net GND1: no longer D1.2 (A), IC1.24 (D), T1.8
- net GND2: now also Q1.1 (S), Q1.2 (S), Q1.3 (S); no longer Q1.5 (D)
- net T2: now also Q1.5 (D); no longer Q1.1 (S), Q1.2 (S), Q1.3 (S)
- new net T8: D1.2 (A), IC1.24 (D), T1.8
Other:
- moved on the sheet: Q1
Changed lines of the file:
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@@
 	)
 	(junction
-		(at 110.49 203.2)
-		(diameter 0)
-		(color 0 0 0 0)
-	)
-	(junction
 		(at 100.33 161.29)
 		(diameter 0)
@@
 	(wire
 		(pts
-			(xy 110.49 203.2) (xy 132.08 203.2)
+			(xy 100.33 203.2) (xy 132.08 203.2)
 		)
 		(stroke
@@
 	(wire
 		(pts
-			(xy 100.33 203.2) (xy 110.49 203.2)
-		)
-		(stroke
-			(width 0)
-			(type default)
-		)
-	)
-	(wire
-		(pts
 			(xy 259.08 99.06) (xy 259.08 93.98)
 		)
@@
 	(wire
 		(pts
-			(xy 110.49 203.2) (xy 110.49 208.28)
-		)
-		(stroke
-			(width 0)
-			(type default)
-		)
-	)
-	(wire
-		(pts
 			(xy 63.5 115.57) (xy 63.5 118.11)
 		)
@@
 		)
 	)
-	(label "T8"
-		(at 110.49 208.28 0)
-		(effects
-			(font
-				(size 1.27 1.27)
-			)
-			(justify left bottom)
-		)
-	)
 	(label "GND1"
 		(at 167.64 167.64 0)
@@
 	(symbol
 		(lib_id "Transistor_FET:FDMS8350LET40")
-		(at 254 83.82 270)
-		(mirror x)
+		(at 254 83.82 90)
 		(unit 1)
 		(body_style 1)
@@
 			)
 		)
-		(property "Value" "100V"
+		(property "Value" "150V"
 			(at 254 77.47 90)
 			(show_name no)
@@
 		)
 		(property "Footprint" "Package_TO_SOT_SMD:TDSON-8-1"
-			(at 252.095 78.74 0)
+			(at 255.905 78.74 0)
 			(hide yes)
 			(show_name no)
@@
 		)
 		(property "Datasheet" "https://www.onsemi.com/pub/Collateral/FDMS8350LET40-D.pdf"
-			(at 250.19 78.74 0)
+			(at 257.81 78.74 0)
 			(hide yes)
 			(show_name no)
