File: flyback1.kicad_pcb (KiCad board)
At the start: 2 copper layers, 52 parts, among them IC1 INN3649C-H606-TL, J1 Conn_02x08_Odd_Even, J2 Conn_02x06_Odd_Even, Q1 100V, T1 P0544NL

Commit message: pcb is organized
Parts:
- added C1: 680p, Capacitor_THT:C_Disc_D8.0mm_W5.0mm_P10.00mm, F.Cu at (207.1, 35.2)
- C2.2: footprint aaa:B58031U9254M062 -> Capacitor_THT:C_Disc_D8.0mm_W5.0mm_P10.00mm
- moved C18 130.5 mm to (230.0, 34.7), turned to -90 degrees
- moved C17 126.6 mm to (227.5, 34.7), turned to -90 degrees
- moved J2 119.1 mm to (235.8, 34.8)
- moved C16 117.0 mm to (224.5, 35.2), turned to -90 degrees
- moved C15 111.5 mm to (221.0, 35.2), turned to -90 degrees
- moved D4 110.2 mm to (216.8, 54.5)
- moved Q1 109.2 mm to (209.4, 66.8), turned to 90 degrees
- moved R1 103.5 mm to (219.8, 86.8), turned to 90 degrees
- moved D1 94.7 mm to (187.2, 66.9), turned to 90 degrees
- moved R15 92.3 mm to (208.5, 91.0), turned to 180 degrees
- moved T1 91.8 mm to (202.5, 73.5), turned to 180 degrees
- moved C8 90.9 mm to (231.0, 61.9)
- moved D5 89.6 mm to (213.5, 92.3), turned to -90 degrees
- moved C10 83.1 mm to (214.5, 86.5), turned to 90 degrees
- moved C11 79.7 mm to (209.3, 86.2), turned to -90 degrees
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Connections:
- C10 pad 1: GND -> /GND2
- C11 pad 2: GND -> /GND2
- C12 pad 1: GND -> /GND2
- C13 pad 2: GND -> /GND2
- C15 pad 2: /OUT2 -> /GND2
- C16 pad 2: /OUT2 -> /GND2
- C17 pad 2: /OUT2 -> /GND2
- C18 pad 2: /OUT2 -> /GND2
- C2.1 pad 1: Net-(J1-Pin_1) -> /T6
- C2.1 pad 2: Net-(J1-Pin_11) -> /GND1
- C2.2 pad 1: Net-(J1-Pin_1) -> /T6
- C2.2 pad 2: Net-(J1-Pin_11) -> /GND1
- C2.3 pad 1: Net-(J1-Pin_1) -> /T6
- C2.3 pad 2: Net-(J1-Pin_11) -> /GND1
- C2.4 pad 1: Net-(J1-Pin_1) -> /T6
- C2.4 pad 2: Net-(J1-Pin_11) -> /GND1
- C5 pad 2: GND -> /GND1
- C6 pad 2: GND -> /GND1
- C7 pad 2: GND -> /GND2
- C8 pad 1: GND -> /GND2
- C9 pad 2: GND -> /GND2
- D1 pad 2: GND -> /GND1
- D5 pad 2: GND -> /GND2
- IC1 pad 16: GND -> /GND1
- IC1 pad 2: GND -> /GND2
- IC1 pad 24: GND -> /GND1
- J1 pad 1: Net-(J1-Pin_1) -> /T6
- J1 pad 11: Net-(J1-Pin_11) -> /GND1
- J1 pad 12: Net-(J1-Pin_11) -> /GND1
- J1 pad 13: Net-(J1-Pin_11) -> /GND1
- J1 pad 14: Net-(J1-Pin_11) -> /GND1
- J1 pad 15: Net-(J1-Pin_11) -> /GND1
- J1 pad 16: Net-(J1-Pin_11) -> /GND1
- J1 pad 2: Net-(J1-Pin_1) -> /T6
- J1 pad 3: Net-(J1-Pin_1) -> /T6
- J1 pad 4: Net-(J1-Pin_1) -> /T6
- J1 pad 5: Net-(J1-Pin_1) -> /T6
- J1 pad 6: Net-(J1-Pin_1) -> /T6
- J2 pad 10: /OUT2 -> /GND2
- J2 pad 11: /OUT2 -> /GND2
- J2 pad 12: /OUT2 -> /GND2
- J2 pad 7: /OUT2 -> /GND2
- J2 pad 8: /OUT2 -> /GND2
- J2 pad 9: /OUT2 -> /GND2
- Q1 pad 5: GND -> /GND2
- R13 pad 2: /OUT2 -> /GND2
- R14 pad 1: GND -> /GND2
- R14 pad 2: /OUT2 -> /GND2
- R16 pad 2: GND -> /GND2
- R2 pad 1: GND -> /GND2
- T1 pad 8: GND -> /GND1
- T1 pad 9: GND -> /GND1
Routing:
- net /+12V: track 0.00 -> 18.4 mm
- net /GND2: track 0.00 -> 12.7 mm

Commit message: tracks drawn
Parts:
- Q1: value 100V -> 150V
- moved C1 21.8 mm to (191.0, 50.0)
- moved R11.1 21.1 mm to (206.6, 50.2)
- moved R11.2 15.8 mm to (206.6, 52.9)
- moved D4 12.1 mm to (206.5, 61.0)
- moved R11.3 11.5 mm to (206.6, 55.6)
- moved C9 11.3 mm to (227.5, 79.2)
- moved C7 10.6 mm to (217.8, 83.2)
- moved R11.4 10.2 mm to (206.6, 58.4)
- moved C13 9.84 mm to (214.9, 66.0)
- moved R16 9.84 mm to (215.0, 70.8)
- moved R2 9.80 mm to (213.8, 83.2)
- moved R1 9.80 mm to (217.5, 77.2)
- moved R14 9.55 mm to (213.7, 88.5)
- moved C10 9.34 mm to (213.5, 77.2), turned to -90 degrees
- moved D5 9.12 mm to (210.8, 83.6)
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Connections:
- D1 pad 2: /GND1 -> /T8
- IC1 pad 24: /GND1 -> /T8
- Q1 pad 1: /T2 -> /GND2
- Q1 pad 2: /T2 -> /GND2
- Q1 pad 3: /T2 -> /GND2
- Q1 pad 5: /GND2 -> /T2
- T1 pad 8: /GND1 -> /T8
Routing:
- net /T6: track 0.00 -> 135.1 mm
- net /+12V: track 18.4 -> 102.6 mm, vias 0 -> 4
- net Net-(D4-A): track 0.00 -> 42.4 mm
- net /T2: track 0.00 -> 38.4 mm
- net /T8: track 0.00 -> 32.6 mm, vias 0 -> 2
- net /BPP: track 0.00 -> 29.9 mm
- net /FB: track 0.00 -> 26.3 mm, vias 0 -> 2
- net Net-(D1-K): track 0.00 -> 25.0 mm
- net Net-(D2-K): track 0.00 -> 24.0 mm
- net /V: track 0.00 -> 21.9 mm
- net Net-(C4-Pad1): track 0.00 -> 20.8 mm
- net /SR: track 0.00 -> 19.3 mm, vias 0 -> 2
- net /BPS: track 0.00 -> 14.2 mm
- net /GND2: track 12.7 -> 0.09 mm, vias 0 -> 21
- net /FWD: track 0.00 -> 10.6 mm
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- added copper zone on B.Cu, net /GND1
- added copper zone on B.Cu, net /GND2
Other:
- board outline added: 123.8 x 63.5 mm

Commit message: finalized pcb
Parts:
- moved R15 0.75 mm to (207.2, 84.2)
Routing:
- net /+12V: track 102.6 -> 125.4 mm, vias 4 -> 6
- net Net-(D5-K): track 0.00 -> 19.8 mm, vias 0 -> 2
- net /GND2: track 0.09 -> 10.2 mm
- net /V: track 21.9 -> 22.6 mm
- net /SR: track 19.3 -> 18.6 mm
- net /FWD: track 10.6 -> 11.2 mm
- net (no net): vias 1 -> 0
Other:
- board size 123.8 x 63.5 mm -> 122.4 x 62.1 mm
