File: _restore_backup_2026-08-25T16-24-23-567/flyback1.kicad_sch (KiCad schematic)
At the start: 52 parts, among them IC1 INN3649C-H606-TL, J1 Conn_02x08_Odd_Even, J2 Conn_02x06_Odd_Even, Q1 100V, T1 P0544NL

Commit message: starting pcb
Parts:
- removed J1: Conn_02x08_Odd_Even, Connector_PinSocket_2.54mm:PinSocket_2x08_P2.54mm_Vertical, symbol Connector_Generic:Conn_02x08_Odd_Even
- removed J2: Conn_02x06_Odd_Even, Connector_PinSocket_2.54mm:PinSocket_2x06_P2.54mm_Vertical, symbol Connector_Generic:Conn_02x06_Odd_Even
- added J1, J2: Conn_01x02_Socket, mpt:MPT0263001TV, symbol Connector:Conn_01x02_Socket
- C2.1: footprint c2.1:C4AQNBW5400M3NJ -> (none)
- C2.2, C2.3, C2.4: footprint aaa:B58031U9254M062 -> (none)
- C8, C9: footprint aaa:16SVF1000M -> (none)
- D1: footprint byg:DIOM5127X229N -> Diode_SMD:D_SMA
- D2: footprint Diode_SMD:D_SMP_DO-220AA -> Diode_THT:D_DO-41_SOD81_P10.16mm_Horizontal
- D3: footprint d3-d4:SOD123_MCC -> Diode_THT:D_DO-41_SOD81_P10.16mm_Horizontal
- D4: footprint d3-d4:SOD123_MCC -> Diode_SMD:D_SMB
- D5: footprint d3-d4:SOD123_MCC -> (none)
- T1: footprint aaa:DIPS1016W120P380L2225H2324Q10N -> Transformer_SMD:Pulse_PA2002NL-PA2008NL-PA2009NL
- VR1: footprint aaa:SOD3716X135N -> (none)
Connections:
- net +12V: now also J2.1 (Pin_1)
- net OUT2: now also J2.2 (Pin_2)
- net at C2.1.1, C2.2.1, C2.3.1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: now also J1.2 (Pin_2)
- net at C2.1.2, C2.2.2, C2.3.2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: now also J1.1 (Pin_1)
- net GND renamed Earth
- no-connect marks 4 -> 0
Other:
- moved on the sheet: C15, C16, C17, C18, C2.1, C2.2, C2.3, C2.4
